File: vibio/pcb-button/vibio-button/vibio-button.kicad_sch (KiCad schematic)
At the start: 1 part

Commit message: Vibio Button PCB
Parts:
- added D1, D2, D3, D4: LED, LED_SMD:LED_1206_3216Metric_Pad1.42x1.75mm_HandSolder, symbol Device:LED
- added J1, J2: Conn_01x03_Female, Connector_PinSocket_2.54mm:PinSocket_1x03_P2.54mm_Vertical, symbol Connector:Conn_01x03_Female
- added R1, R2: R, Resistor_SMD:R_0805_2012Metric_Pad1.20x1.40mm_HandSolder, symbol Device:R
- added R10, R7, R8, R9: 220, Resistor_SMD:R_0805_2012Metric_Pad1.20x1.40mm_HandSolder, symbol Device:R
- added R3, R4, R5, R6: 10k, Resistor_SMD:R_0805_2012Metric_Pad1.20x1.40mm_HandSolder, symbol Device:R
- added SW1, SW2, SW3, SW4: SW_Push, Button_Switch_THT:SW_PUSH-12mm, symbol Switch:SW_Push
- J3: renamed from J?; footprint (none) -> Connector_PinSocket_2.54mm:PinSocket_2x20_P2.54mm_Vertical
Connections:
- net BTN_0: now reaches J3.11 (Pin_11)
- net BTN_0: now also R3.2, SW1.1
- net I2S_SCK: now reaches J3.12 (Pin_12)
- net I2S_SCK: now also J2.3 (Pin_3)
- net BTN_1: now reaches J3.13 (Pin_13)
- net BTN_1: now also R4.2, SW2.1
- net BTN_GND: now reaches J3.14 (Pin_14)
- net BTN_GND: now also SW1.2, SW2.2, SW3.2, SW4.2
- net BTN_2: now reaches J3.15 (Pin_15)
- net BTN_2: now also R5.2, SW3.1
- net BTN_3: now reaches J3.16 (Pin_16)
- net BTN_3: now also R6.2, SW4.1
- net BTN_VDD: now reaches J3.17 (Pin_17)
- net BTN_VDD: now also R3.1, R4.1, R5.1, R6.1
- net LED_0: now reaches J3.3 (Pin_3)
- net LED_0: now also R7.1
- net I2S_WS: now reaches J3.35 (Pin_35)
- net I2S_WS: now also J2.2 (Pin_2)
- net I2S_SD: now reaches J3.38 (Pin_38)
- net I2S_SD: now also J1.3 (Pin_3)
- net LED_GND: now reaches J3.39 (Pin_39)
- net LED_GND: now also D1.1 (K), D2.1 (K), D3.1 (K), D4.1 (K)
- net LED_1: now reaches J3.5 (Pin_5)
- net LED_1: now also R9.1
- net I2S_GND: now reaches J3.6 (Pin_6)
- net I2S_GND: now also J1.1 (Pin_1), R2.1
- net LED_2: now reaches J3.7 (Pin_7)
- net LED_2: now also R10.1
- net LED_3: now reaches J3.9 (Pin_9)
- net LED_3: now also R8.1
- net VDD renamed I2S_VDD
- net I2S_VDD: now also J1.2 (Pin_2), R1.1
- new net: D3.2 (A), R9.2
- new net: D1.2 (A), R7.2
- new net: D4.2 (A), R10.2
- new net: D2.2 (A), R8.2
- new net I2S_LR: J2.1 (Pin_1), R1.2, R2.2
Other:
- moved on the sheet: J3
