File: recruitmen/formulatrix/logic_driver/logic_driver.kicad_pcb (KiCad board)
At the start: 2 copper layers, 68.5 x 33.9 mm, 16 parts, among them J1 Sensor Input, J2 Sensor Input, J3 Motor Output, J4 Conn_01x02_Socket, J5 Conn_01x02_Socket, Q1 IRG4PF50W, U1 LM358_DFN, U2 4070, U3 4N35, U4 L7805

Commit message: PCB Recruitment
Parts:
- added D2: D, Diode_THT:D_A-405_P7.62mm_Horizontal, F.Cu at (79.2, 80.0)
- moved J3 2.31 mm to (70.6, 71.5)
Routing:
- net Net-(D2-K): track 11.5 -> 18.8 mm
- net MTRPWR: track 18.3 -> 20.6 mm
Changed lines of the file:
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@@
   (net 3 "Net-(J2-Pin_1)")
   (net 4 "MTRPWR")
-  (net 5 "Net-(J3-Pin_2)")
+  (net 5 "Net-(D2-K)")
   (net 6 "+15V")
   (net 7 "GNDPWR")
@@
   )
   (footprint "TerminalBlock:TerminalBlock_Altech_AK300-2_P5.00mm" (layer "F.Cu")
-    (at 72.88 71.35 -90)
+    (at 70.57 71.45 -90)
     (descr "Altech AK300 terminal block, pitch 5.0mm, 45 degree angled, see http://www.mouser.com/ds/2/16/PCBMETRC-24178.pdf")
     (tags "Altech AK300 terminal block pitch 5.0mm")
@@
       (net 4 "MTRPWR") (pinfunction "Pin_1") (pintype "passive"))
     (pad "2" thru_hole oval (at 5 0 270) (size 1.98 3.96) (drill 1.32) (layers "*.Cu" "*.Mask")
-      (net 5 "Net-(J3-Pin_2)") (pinfunction "Pin_2") (pintype "passive"))
+      (net 5 "Net-(D2-K)") (pinfunction "Pin_2") (pintype "passive"))
     (model "${KICAD6_3DMODEL_DIR}/TerminalBlock.3dshapes/TerminalBlock_Altech_AK300-2_P5.00mm.wrl"
       (offset (xyz 0 0 0))
@@
     (pad "1" smd circle (at 0 0) (size 4 4) (layers "F.Cu" "F.Mask")
       (net 10 "Net-(U1A--)") (pinfunction "1") (pintype "passive"))
+  )
+  (footprint "Diode_THT:D_A-405_P7.62mm_Horizontal" (layer "F.Cu")
+    (at 79.19 80.02 90)
+    (descr "Diode, A-405 series, Axial, Horizontal, pin pitch=7.62mm, , length*diameter=5.2*2.7mm^2, , http://www.diodes.com/_files/packages/A-405.pdf")
+    (tags "Diode A-405 series Axial Horizontal pin pitch 7.62mm  length 5.2mm diameter 2.7mm")
+    (property "Sheetfile" "logic_driver.kicad_sch")
+    (property "Sheetname" "")
+    (property "Sim.Device" "D")
+    (property "Sim.Pins" "1=K 2=A")
+    (property "ki_description" "Diode")
+    (property "ki_keywords" "diode")
+    (attr through_hole)
+    (fp_text reference "D2" (at 3.81 -2.47 90) (layer "F.SilkS")
+        (effects (font (size 1 1) (thickness 0.15)))
+    )
+    (fp_text value "D" (at 3.81 2.47 90) (layer "F.Fab")
+        (effects (font (size 1 1) (thickness 0.15)))
+    )
+    (fp_text user "K" (at 0 -1.9 90) (layer "F.SilkS")
+        (effects (font (size 1 1) (thickness 0.15)))
+    )
+    (fp_text user "K" (at 0 -1.9 90) (layer "F.Fab")
+        (effects (font (size 1 1) (thickness 0.15)))
+    )
+    (fp_text user "${REFERENCE}" (at 4.2 0 90) (layer "F.Fab")
+        (effects (font (size 1 1) (thickness 0.15)))
+    )
+    (fp_line (start 1.09 -1.47) (end 6.53 -1.47)
+      (stroke (width 0.12) (type solid)) (layer "F.SilkS"))
+    (fp_line (start 1.09 -1.14) (end 1.09 -1.47)
+      (stroke (width 0.12) (type solid)) (layer "F.SilkS"))
+    (fp_line (start 1.09 1.14) (end 1.09 1.47)
+      (stroke (width 0.12) (type solid)) (layer "F.SilkS"))
+    (fp_line (start 1.09 1.47) (end 6.53 1.47)
+      (stroke (width 0.12) (type solid)) (layer "F.SilkS"))
+    (fp_line (start 1.87 -1.47) (end 1.87 1.47)
+      (stroke (width 0.12) (type solid)) (layer "F.SilkS"))
+    (fp_line (start 1.99 -1.47) (end 1.99 1.47)
+      (stroke (width 0.12) (type solid)) (layer "F.SilkS"))
+    (fp_line (start 2.11 -1.47) (end 2.11 1.47)
+      (stroke (width 0.12) (type solid)) (layer "F.SilkS"))
+    (fp_line (start 6.53 -1.47) (end 6.53 -1.14)
+      (stroke (width 0.12) (type solid)) (layer "F.SilkS"))
+    (fp_line (start 6.53 1.47) (end 6.53 1.14)
+      (stroke (width 0.12) (type solid)) (layer "F.SilkS"))
+    (fp_line (start -1.15 -1.6) (end -1.15 1.6)
+      (stroke (width 0.05) (type solid)) (layer "F.CrtYd"))
+    (fp_line (start -1.15 1.6) (end 8.77 1.6)
+      (stroke (width 0.05) (type solid)) (layer "F.CrtYd"))
+    (fp_line (start 8.77 -1.6) (end -1.15 -1.6)
+      (stroke (width 0.05) (type solid)) (layer "F.CrtYd"))
+    (fp_line (start 8.77 1.6) (end 8.77 -1.6)
+      (stroke (width 0.05) (type solid)) (layer "F.CrtYd"))
+    (fp_line (start 0 0) (end 1.21 0)
+      (stroke (width 0.1) (type solid)) (layer "F.Fab"))
+    (fp_line (start 1.21 -1.35) (end 1.21 1.35)
+      (stroke (width 0.1) (type solid)) (layer "F.Fab"))
+    (fp_line (start 1.21 1.35) (end 6.41 1.35)
+      (stroke (width 0.1) (type solid)) (layer "F.Fab"))
+    (fp_line (start 1.89 -1.35) (end 1.89 1.35)
+      (stroke (width 0.1) (type solid)) (layer "F.Fab"))
+    (fp_line (start 1.99 -1.35) (end 1.99 1.35)
+      (stroke (width 0.1) (type solid)) (layer "F.Fab"))
+    (fp_line (start 2.09 -1.35) (end 2.09 1.35)
+      (stroke (width 0.1) (type solid)) (layer "F.Fab"))
+    (fp_line (start 6.41 -1.35) (end 1.21 -1.35)
+      (stroke (width 0.1) (type solid)) (layer "F.Fab"))
+    (fp_line (start 6.41 1.35) (end 6.41 -1.35)
+      (stroke (width 0.1) (type solid)) (layer "F.Fab"))
+    (fp_line (start 7.62 0) (end 6.41 0)
+      (stroke (width 0.1) (type solid)) (layer "F.Fab"))
+    (pad "1" thru_hole rect (at 0 0 90) (size 1.8 1.8) (drill 0.9) (layers "*.Cu" "*.Mask")
+      (net 5 "Net-(D2-K)") (pinfunction "K") (pintype "passive"))
+    (pad "2" thru_hole oval (at 7.62 0 90) (size 1.8 1.8) (drill 0.9) (layers "*.Cu" "*.Mask")
+      (net 7 "GNDPWR") (pinfunction "A") (pintype "passive"))
+    (model "${KICAD6_3DMODEL_DIR}/Diode_THT.3dshapes/D_A-405_P7.62mm_Horizontal.wrl"
+      (offset (xyz 0 0 0))
+      (scale (xyz 1 1 1))
+      (rotate (xyz 0 0 0))
+    )
   )
   (footprint "Package_DFN_QFN:DFN-8-1EP_2x2mm_P0.5mm_EP1.05x1.75mm" (layer "F.Cu")
@@
       (net 8 "Net-(Q1-G)") (pinfunction "G") (pintype "input"))
     (pad "2" thru_hole oval (at 5.45 0 90) (size 2.5 4.5) (drill 1.5) (layers "*.Cu" "*.Mask")
-      (net 5 "Net-(J3-Pin_2)") (pinfunction "C") (pintype "passive"))
+      (net 5 "Net-(D2-K)") (pinfunction "C") (pintype "passive"))
     (pad "3" thru_hole oval (at 10.9 0 90) (size 2.5 4.5) (drill 1.5) (layers "*.Cu" "*.Mask")
       (net 7 "GNDPWR") (pinfunction "E") (pintype "passive"))
@@
   (segment (start 127.86 61.39) (end 125.42 58.95) (width 0.5) (layer "B.Cu") (net 3))
   (segment (start 127.86 71.7) (end 127.86 61.39) (width 0.5) (layer "B.Cu") (net 3))
-  (segment (start 75.41 71.35) (end 72.88 71.35) (width 2) (layer "B.Cu") (net 4))
-  (segment (start 77.6 69.16) (end 75.41 71.35) (width 2) (layer "B.Cu") (net 4))
+  (segment (start 75.31 71.45) (end 70.57 71.45) (width 2) (layer "B.Cu") (net 4))
+  (segment (start 77.6 69.16) (end 75.31 71.45) (width 2) (layer "B.Cu") (net 4))
   (segment (start 77.6 56.51) (end 77.6 69.16) (width 2) (layer "B.Cu") (net 4))
-  (segment (start 82.74 76.35) (end 83.92 75.17) (width 2) (layer "B.Cu") (net 5))
-  (segment (start 72.88 76.35) (end 82.74 76.35) (width 2) (layer "B.Cu") (net 5))
+  (segment (start 79 75.17) (end 77.93 75.17) (width 2) (layer "B.Cu") (net 5))
+  (segment (start 79.19 80.02) (end 79.19 75.36) (width 2) (layer "B.Cu") (net 5))
+  (segment (start 76.65 76.45) (end 70.57 76.45) (width 2) (layer "B.Cu") (net 5))
+  (segment (start 83.92 75.17) (end 79 75.17) (width 2) (layer "B.Cu") (net 5))
+  (segment (start 77.93 75.17) (end 76.65 76.45) (width 2) (layer "B.Cu") (net 5))
+  (segment (start 79.19 75.36) (end 79 75.17) (width 2) (layer "B.Cu") (net 5))
   (segment (start 87.19 62.08) (end 86.45 61.34) (width 1) (layer "F.Cu") (net 6))
   (segment (start 100.35 62.08) (end 87.19 62.08) (width 1) (layer "F.Cu") (net 6))
