File: halogen-flicker/circuit/halodc_flicker_v0/halodc_flicker_v0.kicad_pcb (KiCad board)
At the start: 2 copper layers, 86.1 x 45.6 mm, 21 parts, among them J1 ASP, J2 BATT_LAMP, J4 CHARGER, Q1 IRF540N, SW1 SW_DIP_x02, SW2 SW_Push, U1 ATtiny13A-S, U2 PC817, U3 AMS1117-5.0

Commit message: Halogen Flicker
Parts:
- moved Q1 40.1 mm to (101.8, 65.3)
- moved C1 40.1 mm to (128.5, 51.6)
- moved C2 40.1 mm to (140.6, 57.8)
- moved C3 40.1 mm to (95.4, 58.4)
- moved D1 40.1 mm to (124.2, 45.9)
- moved D3 40.1 mm to (125.1, 66.1)
- moved H1 40.1 mm to (154.3, 45.2)
- moved H2 40.1 mm to (78.8, 45.0)
- moved J1 40.1 mm to (137.5, 57.8)
- moved J2 40.1 mm to (117.7, 75.2)
- moved J4 40.1 mm to (142.6, 66.5)
- moved R1 40.1 mm to (120.5, 65.0)
- moved R2 40.1 mm to (108.0, 65.0)
- moved R3 40.1 mm to (124.2, 48.0)
- moved R4 40.1 mm to (125.1, 63.9)
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
Commit message: Halogen Flicker
Routing:
- net GNDPWR: track 128.1 -> 125.6 mm
- net +12V: track 57.3 -> 58.9 mm
Changed lines of the file:
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@@
       (layerselection 0x00010fc_ffffffff)
       (plot_on_all_layers_selection 0x0000000_00000000)
-      (disableapertmacros false)
+      (disableapertmacros true)
       (usegerberextensions false)
       (usegerberattributes true)
@@
       (svgprecision 4)
       (plotframeref false)
-      (viasonmask false)
+      (viasonmask true)
       (mode 1)
-      (useauxorigin false)
+      (useauxorigin true)
       (hpglpennumber 1)
       (hpglpenspeed 20)
@@
       (plotinvisibletext false)
       (sketchpadsonfab false)
-      (subtractmaskfromsilk false)
+      (subtractmaskfromsilk true)
       (outputformat 1)
       (mirror false)
-      (drillshape 1)
+      (drillshape 0)
       (scaleselection 1)
-      (outputdirectory "")
+      (outputdirectory "exports/gerber/")
     )
   )
@@
     (property "ki_keywords" "R res resistor")
     (attr smd)
-    (fp_text reference "R2" (at 0 -1.65 90) (layer "F.SilkS")
+    (fp_text reference "R2" (at 2.985 -0.03 90) (layer "F.SilkS")
         (effects (font (size 1 1) (thickness 0.15)))
     )
@@
   (segment (start 94.405 58.41) (end 94.405 54.185) (width 1.5) (layer "F.Cu") (net 2))
   (segment (start 94.405 54.185) (end 95.18 53.41) (width 1.5) (layer "F.Cu") (net 2))
-  (via (at 119.55 58.55) (size 2) (drill 0.6) (layers "F.Cu" "B.Cu") (net 2))
-  (via (at 127.35 45.95) (size 2) (drill 0.6) (layers "F.Cu" "B.Cu") (net 2))
-  (via (at 125.35 51.45) (size 2) (drill 0.6) (layers "F.Cu" "B.Cu") (net 2))
-  (via (at 99.35 52.45) (size 2) (drill 0.6) (layers "F.Cu" "B.Cu") (net 2))
+  (via (at 119.55 58.55) (size 2) (drill 0.7) (layers "F.Cu" "B.Cu") (net 2))
+  (via (at 127.35 45.95) (size 2) (drill 0.7) (layers "F.Cu" "B.Cu") (net 2))
+  (via (at 125.35 51.45) (size 2) (drill 0.7) (layers "F.Cu" "B.Cu") (net 2))
+  (via (at 99.35 52.45) (size 2) (drill 0.7) (layers "F.Cu" "B.Cu") (net 2))
   (segment (start 96.48 58.41) (end 96.49 58.41) (width 1.5) (layer "F.Cu") (net 3))
   (segment (start 105.78 57.61) (end 105.78 47.42) (width 2) (layer "F.Cu") (net 3))
@@
   (segment (start 86.29 53.41) (end 84.65 55.05) (width 2) (layer "F.Cu") (net 5))
   (segment (start 94.06 62.65) (end 96.69 65.28) (width 2) (layer "F.Cu") (net 5))
-  (via (at 85.15 76.45) (size 2) (drill 0.6) (layers "F.Cu" "B.Cu") (net 5))
+  (via (at 85.15 76.45) (size 2) (drill 0.7) (layers "F.Cu" "B.Cu") (net 5))
   (segment (start 110.6 80.95) (end 126.3 80.95) (width 2) (layer "B.Cu") (net 5))
   (segment (start 127.65 79.6) (end 127.65 75.25) (width 2) (layer "B.Cu") (net 5))
@@
   (segment (start 117.35 59.55) (end 118.45 60.65) (width 0.7) (layer "F.Cu") (net 6))
   (segment (start 117.35 55.15) (end 117.35 59.55) (width 0.7) (layer "F.Cu") (net 6))
-  (via (at 128.45 65.85) (size 2) (drill 0.6) (layers "F.Cu" "B.Cu") (net 6))
-  (via (at 122.85 60.25) (size 2) (drill 0.6) (layers "F.Cu" "B.Cu") (net 6))
+  (via (at 128.45 65.85) (size 2) (drill 0.7) (layers "F.Cu" "B.Cu") (net 6))
+  (via (at 122.85 60.25) (size 2) (drill 0.7) (layers "F.Cu" "B.Cu") (net 6))
   (segment (start 125.45 60.25) (end 128.05 62.85) (width 0.7) (layer "B.Cu") (net 6))
   (segment (start 122.85 60.25) (end 125.45 60.25) (width 0.7) (layer "B.Cu") (net 6))
@@
   (segment (start 124.095 63.92) (end 124.095 66.075) (width 0.7) (layer "F.Cu") (net 7))
   (segment (start 124.095 66.075) (end 124.105 66.085) (width 0.7) (layer "F.Cu") (net 7))
-  (segment (start 78.75 44.95) (end 78.75 66.75) (width 5) (layer "B.Cu") (net 8))
-  (segment (start 78.75 66.75) (end 81.85 69.85) (width 5) (layer "B.Cu") (net 8))
-  (segment (start 129.852999 71.245) (end 129.074295 70.466296) (width 5) (layer "B.Cu") (net 8))
-  (segment (start 154.35 66.75) (end 149.855 71.245) (width 5) (layer "B.Cu") (net 8))
-  (segment (start 129.074295 70.466296) (end 107.266295 70.466296) (width 5) (layer "B.Cu") (net 8))
-  (segment (start 81.85 69.85) (end 97.71 69.85) (width 5) (layer "B.Cu") (net 8))
-  (segment (start 154.35 45.2) (end 154.35 66.75) (width 5) (layer "B.Cu") (net 8))
+  (segment (start 151 70.75) (end 154.35 67.4) (width 4) (layer "B.Cu") (net 8))
+  (segment (start 86.55 70.75) (end 151 70.75) (width 4) (layer "B.Cu") (net 8))
+  (segment (start 78.75 44.95) (end 78.75 62.95) (width 4) (layer "B.Cu") (net 8))
   (segment (start 99.23 65.28) (end 99.23 68.33) (width 2) (layer "B.Cu") (net 8))
-  (segment (start 107.266295 70.466296) (end 106.982591 70.75) (width 5) (layer "B.Cu") (net 8))
-  (segment (start 149.855 71.245) (end 129.852999 71.245) (width 5) (layer "B.Cu") (net 8))
+  (segment (start 78.75 62.95) (end 86.55 70.75) (width 4) (layer "B.Cu") (net 8))
   (segment (start 99.23 68.33) (end 97.71 69.85) (width 2) (layer "B.Cu") (net 8))
-  (segment (start 98.61 70.75) (end 97.71 69.85) (width 5) (layer "B.Cu") (net 8))
-  (segment (start 106.982591 70.75) (end 98.61 70.75) (width 5) (layer "B.Cu") (net 8))
+  (segment (start 154.35 67.4) (end 154.35 45.2) (width 4) (layer "B.Cu") (net 8))
   (segment (start 133.29 57.84) (end 135 57.84) (width 0.7) (layer "F.Cu") (net 9))
   (segment (start 129.38 56.445) (end 131.895 56.445) (width 0.7) (layer "F.Cu") (net 9))
@@
   (segment (start 133.9 60.8) (end 134.3 60.8) (width 0.7) (layer "F.Cu") (net 10))
   (segment (start 130.815 57.715) (end 131.95 58.85) (width 0.7) (layer "F.Cu") (net 10))
-  (via (at 134.3 60.8) (size 2) (drill 0.6) (layers "F.Cu" "B.Cu") (net 10))
+  (via (at 134.3 60.8) (size 2) (drill 0.7) (layers "F.Cu" "B.Cu") (net 10))
   (segment (start 139.85 55.35) (end 139.8 55.3) (width 0.7) (layer "B.Cu") (net 10))
   (segment (start 139.8 55.3) (end 137.54 55.3) (width 0.7) (layer "B.Cu") (net 10))
@@
   (segment (start 127.35 60.3) (end 130 60.3) (width 0.7) (layer "F.Cu") (net 12))
   (segment (start 122.08 53.905) (end 125.555 53.905) (width 0.7) (layer "F.Cu") (net 12))
-  (via (at 131.15 61.45) (size 2) (drill 0.6) (layers "F.Cu" "B.Cu") (net 12))
+  (via (at 131.15 61.45) (size 2) (drill 0.7) (layers "F.Cu" "B.Cu") (net 12))
   (segment (start 131.15 61.45) (end 131.15 56.61) (width 0.7) (layer "B.Cu") (net 12))
   (segment (start 131.15 56.61) (end 135 52.76) (width 0.7) (layer "B.Cu") (net 12))
@@
   (segment (start 122.65 73.15) (end 122.65 75.25) (width 2) (layer "F.Cu") (net 13))
   (segment (start 105.45 67.05) (end 109.95 71.55) (width 1.5) (layer "F.Cu") (net 13))
-  (via (at 105.45 65.7) (size 2) (drill 0.6) (layers "F.Cu" "B.Cu") (net 13))
-  (via (at 97.45 61.65) (size 2) (drill 0.6) (layers "F.Cu" "B.Cu") (net 13))
-  (segment (start 97.45 61.65) (end 101.436004 61.65) (width 1.5) (layer "B.Cu") (net 13))
-  (segment (start 101.436004 61.65) (end 105.45 65.663996) (width 1.5) (layer "B.Cu") (net 13))
+  (via (at 105.45 65.7) (size 2) (drill 0.7) (layers "F.Cu" "B.Cu") (net 13))
+  (via (at 97.45 61.65) (size 2) (drill 0.7) (layers "F.Cu" "B.Cu") (net 13))
+  (segment (start 105.35 62.85) (end 105.35 65.6) (width 2) (layer "B.Cu") (net 13))
+  (segment (start 97.45 61.65) (end 104.15 61.65) (width 2) (layer "B.Cu") (net 13))
   (segment (start 105.45 65.663996) (end 105.45 65.7) (width 2) (layer "B.Cu") (net 13))
+  (segment (start 105.35 65.6) (end 105.45 65.7) (width 2) (layer "B.Cu") (net 13))
+  (segment (start 104.15 61.65) (end 105.35 62.85) (width 2) (layer "B.Cu") (net 13))
   (segment (start 110.51 62.01) (end 109.75 61.25) (width 1.5) (layer "F.Cu") (net 16))
   (segment (start 109.75 61.25) (end 103.55 61.25) (width 1.5) (layer "F.Cu") (net 16))

Commit message: Update PCB FLicker Halogen
Parts:
- removed C1, C2, C3: 100nF, Capacitor_SMD:C_0805_2012Metric_Pad1.18x1.45mm_HandSolder
- removed SW2: SW_Push, Button_Switch_THT:SW_Tactile_SPST_Angled_PTS645Vx31-2LFS
- removed U1: ATtiny13A-S, Package_SO:SOIC-8W_5.3x5.3mm_P1.27mm
- added J3: SW_ON, Connector_PinSocket_2.54mm:PinSocket_1x02_P2.54mm_Vertical, F.Cu at (121.2, 54.5)
- added U4: ATtiny13A-P, Package_DIP:DIP-8_W7.62mm, F.Cu at (123.0, 59.5)
- D1, D3, R1, R2, R3, R4, U3: moved to B.Cu
- D2: footprint Diode_SMD:D_SMB-SMC_Universal_Handsoldering -> Diode_SMD:D_SMA-SMB_Universal_Handsoldering; moved to B.Cu
- moved R3 22.1 mm to (144.0, 57.8), turned to 90 degrees
- moved D1 20.1 mm to (140.9, 57.0), turned to 0 degrees
- moved R1 17.9 mm to (102.7, 66.5), turned to 180 degrees
- moved U2 16.7 mm to (101.7, 68.8), turned to -90 degrees
- moved Q1 13.2 mm to (94.8, 76.5), turned to 90 degrees
- moved R4 11.7 mm to (114.0, 67.5)
- moved R2 11.4 mm to (104.4, 75.8)
- moved D3 11.2 mm to (114.0, 65.6)
- moved J1 7.49 mm to (139.9, 65.0)
- moved D2 7.28 mm to (92.8, 60.6), turned to -90 degrees
- moved SW1 7.14 mm to (107.0, 59.2)
- moved J4 6.55 mm to (143.8, 72.9)
- moved U3 3.87 mm to (100.0, 60.5)
- moved J2 3.17 mm to (119.7, 77.7)
- moved H1 0.62 mm to (154.2, 44.6)
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Routing:
- net +12V: track 58.9 -> 195.6 mm, vias 2 -> 0
- net GND: track 25.8 -> 102.5 mm
- net Net-(D3-K): track 22.4 -> 3.98 mm, vias 2 -> 0
- net SEL: track 7.78 -> 25.3 mm
- net +5V: track 65.2 -> 54.7 mm, vias 0 -> 4
- net GNDREF: track 108.5 -> 98.1 mm, vias 1 -> 2
- net CON: track 18.4 -> 28.2 mm
- net Net-(Q1-G): track 13.5 -> 4.40 mm
- net GNDPWR: track 125.6 -> 117.1 mm
- net MOSI: track 18.9 -> 25.0 mm, vias 1 -> 0
- net SCK: track 5.67 -> 6.88 mm
- net NRST: track 25.2 -> 26.0 mm, vias 1 -> 2
- net MISO: track 6.20 -> 6.88 mm
- net Net-(J3-Pin_1): track 29.9 -> 29.3 mm
- added copper zone on B.Cu, net (none)
- removed copper zone on F.Cu, net (none)
- removed copper zone on B.Cu, net GND
- removed copper zone on B.Cu, net GNDREF
Other:
- board size 86.1 x 45.6 mm -> 86.1 x 48.6 mm

Commit message: Update PCB FLicker
Routing:
- added copper zone on F.Cu, net (none)
Changed lines of the file:
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@@
     (fp_line (start 8.89 2.88) (end 8.89 -2.92)
       (stroke (width 0.1) (type solid)) (layer "F.Fab"))
-    (pad "1" thru_hole roundrect (at 0 0 180) (size 1.74 2.19) (drill 1.19) (layers "*.Cu" "*.Mask") (roundrect_rratio 0.143678)
+    (pad "1" thru_hole roundrect (at 0 0 180) (size 1.74 2.19) (drill 1.19) (layers "*.Cu" "*.Mask") (roundrect_rratio 0.1436781609)
       (net 5 "GNDREF") (pinfunction "Pin_1") (pintype "passive"))
     (pad "2" thru_hole oval (at 2.54 0 180) (size 1.74 2.19) (drill 1.19) (layers "*.Cu" "*.Mask")
@@
     (fp_line (start 1 0.625) (end 1 -0.625)
       (stroke (width 0.1) (type solid)) (layer "B.Fab"))
-    (pad "1" smd roundrect (at -1 0 90) (size 1.2 1.4) (layers "B.Cu" "B.Paste" "B.Mask") (roundrect_rratio 0.208333)
+    (pad "1" smd roundrect (at -1 0 90) (size 1.2 1.4) (layers "B.Cu" "B.Paste" "B.Mask") (roundrect_rratio 0.2083333333)
       (net 1 "+5V") (pintype "passive"))
-    (pad "2" smd roundrect (at 1 0 90) (size 1.2 1.4) (layers "B.Cu" "B.Paste" "B.Mask") (roundrect_rratio 0.208333)
+    (pad "2" smd roundrect (at 1 0 90) (size 1.2 1.4) (layers "B.Cu" "B.Paste" "B.Mask") (roundrect_rratio 0.2083333333)
       (net 4 "Net-(D1-A)") (pintype "passive"))
     (model "${KICAD6_3DMODEL_DIR}/Resistor_SMD.3dshapes/R_0805_2012Metric.wrl"
@@
     (fp_line (start 1 0.625) (end 1 -0.625)
       (stroke (width 0.1) (type solid)) (layer "B.Fab"))
-    (pad "1" smd roundrect (at -1 0) (size 1.2 1.4) (layers "B.Cu" "B.Paste" "B.Mask") (roundrect_rratio 0.208333)
+    (pad "1" smd roundrect (at -1 0) (size 1.2 1.4) (layers "B.Cu" "B.Paste" "B.Mask") (roundrect_rratio 0.2083333333)
       (net 7 "Net-(D3-A)") (pintype "passive"))
-    (pad "2" smd roundrect (at 1 0) (size 1.2 1.4) (layers "B.Cu" "B.Paste" "B.Mask") (roundrect_rratio 0.208333)
+    (pad "2" smd roundrect (at 1 0) (size 1.2 1.4) (layers "B.Cu" "B.Paste" "B.Mask") (roundrect_rratio 0.2083333333)
       (net 17 "CON") (pintype "passive"))
     (model "${KICAD6_3DMODEL_DIR}/Resistor_SMD.3dshapes/R_0805_2012Metric.wrl"
@@
     (fp_line (start 1 0.6) (end -0.7 0.6)
       (stroke (width 0.1) (type solid)) (layer "B.Fab"))
-    (pad "1" smd roundrect (at -1.025 0) (size 1.15 1.4) (layers "B.Cu" "B.Paste" "B.Mask") (roundrect_rratio 0.217391)
+    (pad "1" smd roundrect (at -1.025 0) (size 1.15 1.4) (layers "B.Cu" "B.Paste" "B.Mask") (roundrect_rratio 0.2173913043)
       (net 2 "GND") (pinfunction "K") (pintype "passive"))
-    (pad "2" smd roundrect (at 1.025 0) (size 1.15 1.4) (layers "B.Cu" "B.Paste" "B.Mask") (roundrect_rratio 0.217391)
+    (pad "2" smd roundrect (at 1.025 0) (size 1.15 1.4) (layers "B.Cu" "B.Paste" "B.Mask") (roundrect_rratio 0.2173913043)
       (net 4 "Net-(D1-A)") (pinfunction "A") (pintype "passive"))
     (model "${KICAD6_3DMODEL_DIR}/LED_SMD.3dshapes/LED_0805_2012Metric.wrl"
@@
     (fp_line (start 1 0.6) (end -0.7 0.6)
       (stroke (width 0.1) (type solid)) (layer "B.Fab"))
-    (pad "1" smd roundrect (at -1.025 0 180) (size 1.15 1.4) (layers "B.Cu" "B.Paste" "B.Mask") (roundrect_rratio 0.217391)
+    (pad "1" smd roundrect (at -1.025 0 180) (size 1.15 1.4) (layers "B.Cu" "B.Paste" "B.Mask") (roundrect_rratio 0.2173913043)
       (net 6 "Net-(D3-K)") (pinfunction "K") (pintype "passive"))
-    (pad "2" smd roundrect (at 1.025 0 180) (size 1.15 1.4) (layers "B.Cu" "B.Paste" "B.Mask") (roundrect_rratio 0.217391)
+    (pad "2" smd roundrect (at 1.025 0 180) (size 1.15 1.4) (layers "B.Cu" "B.Paste" "B.Mask") (roundrect_rratio 0.2173913043)
       (net 7 "Net-(D3-A)") (pinfunction "A") (pintype "passive"))
     (model "${KICAD6_3DMODEL_DIR}/LED_SMD.3dshapes/LED_0805_2012Metric.wrl"
@@
     (fp_line (start 1 0.625) (end 1 -0.625)
       (stroke (width 0.1) (type solid)) (layer "B.Fab"))
-    (pad "1" smd roundrect (at -1 0 180) (size 1.2 1.4) (layers "B.Cu" "B.Paste" "B.Mask") (roundrect_rratio 0.208333)
+    (pad "1" smd roundrect (at -1 0 180) (size 1.2 1.4) (layers "B.Cu" "B.Paste" "B.Mask") (roundrect_rratio 0.2083333333)
       (net 17 "CON") (pintype "passive"))
-    (pad "2" smd roundrect (at 1 0 180) (size 1.2 1.4) (layers "B.Cu" "B.Paste" "B.Mask") (roundrect_rratio 0.208333)
+    (pad "2" smd roundrect (at 1 0 180) (size 1.2 1.4) (layers "B.Cu" "B.Paste" "B.Mask") (roundrect_rratio 0.2083333333)
       (net 18 "Net-(R1-Pad2)") (pintype "passive"))
     (model "${KICAD6_3DMODEL_DIR}/Resistor_SMD.3dshapes/R_0805_2012Metric.wrl"
@@
     (fp_line (start 1 0.625) (end 1 -0.625)
       (stroke (width 0.1) (type solid)) (layer "B.Fab"))
-    (pad "1" smd roundrect (at -1 0 90) (size 1.2 1.4) (layers "B.Cu" "B.Paste" "B.Mask") (roundrect_rratio 0.208333)
+    (pad "1" smd roundrect (at -1 0 90) (size 1.2 1.4) (layers "B.Cu" "B.Paste" "B.Mask") (roundrect_rratio 0.2083333333)
       (net 19 "Net-(R2-Pad1)") (pintype "passive"))
-    (pad "2" smd roundrect (at 1 0 90) (size 1.2 1.4) (layers "B.Cu" "B.Paste" "B.Mask") (roundrect_rratio 0.208333)
+    (pad "2" smd roundrect (at 1 0 90) (size 1.2 1.4) (layers "B.Cu" "B.Paste" "B.Mask") (roundrect_rratio 0.2083333333)
       (net 13 "+12V") (pintype "passive"))
     (model "${KICAD6_3DMODEL_DIR}/Resistor_SMD.3dshapes/R_0805_2012Metric.wrl"
@@
   (segment (start 125.12 64.53) (end 128.55 61.1) (width 0.7) (layer "B.Cu") (net 20))
   (segment (start 123 64.53) (end 125.12 64.53) (width 0.7) (layer "B.Cu") (net 20))
+  (zone (net 0) (net_name "") (layer "F.Cu") (hatch edge 0.5)
+    (priority 1)
+    (connect_pads (clearance 1))
+    (min_thickness 0.25) (filled_areas_thickness no)
+    (fill yes (thermal_gap 0.5) (thermal_bridge_width 0.5) (island_removal_mode 1) (island_area_min 10))
+    (polygon
+      (pts
+        (xy 73.3 39.35)
+        (xy 159.45 39.55)
+        (xy 159.5 88.1)
+        (xy 73.4 88.05)
+      )
+    )
+  )
   (zone (net 0) (net_name "") (layer "B.Cu") (hatch edge 0.5)
     (connect_pads (clearance 1.5))

Commit message: Halogen and ATTiny is hard
Parts:
- R1: value 100 -> 10K
Changed lines of the file:
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@@
         (effects (font (size 1 1) (thickness 0.15)) (justify mirror))
     )
-    (fp_text value "100" (at 0 -1.65) (layer "B.Fab")
+    (fp_text value "10K" (at 0 -1.65) (layer "B.Fab")
         (effects (font (size 1 1) (thickness 0.15)) (justify mirror))
     )
