File: halogen-flicker/circuit/halodc_flicker_v0/halodc_flicker_v0.kicad_sch (KiCad schematic)
At the start: 21 parts, among them J1 SPI, J2 Conn_01x02_Pin, J3 Conn_01x02_Pin, Q1 IRF540N, SW1 SW_DIP_x02, SW2 SW_Push, U1 ATtiny13A-S, U2 PC817, U3 AMS1117-5.0

Commit message: Halogen FLicker
Parts:
- removed J2, J3: Conn_01x02_Pin, symbol Connector:Conn_01x02_Pin
- added J2: BATT_LAMP, TerminalBlock:TerminalBlock_Altech_AK300-3_P5.00mm, symbol Connector:Conn_01x03_Pin
- added J4: CHARGER, Connector_Molex:Molex_KK-254_AE-6410-04A_1x04_P2.54mm_Vertical, symbol Connector:Conn_01x04_Pin
- C1, C2, C3: value 10nF -> 100nF; footprint (none) -> Capacitor_SMD:C_0805_2012Metric_Pad1.18x1.45mm_HandSolder
- D1, D3: footprint (none) -> LED_SMD:LED_0805_2012Metric_Pad1.15x1.40mm_HandSolder
- D2: footprint (none) -> Diode_SMD:D_SMB-SMC_Universal_Handsoldering
- H1, H2: footprint (none) -> MountingHole:MountingHole_4.5mm_Pad
- J1: value SPI -> ASP; footprint (none) -> Connector_PinHeader_2.54mm:PinHeader_2x03_P2.54mm_Vertical
- Q1: footprint Package_TO_SOT_THT:TO-220-3_Vertical -> Package_TO_SOT_THT:TO-220-3_Horizontal_TabDown
- R1, R2, R3, R4: footprint (none) -> Resistor_SMD:R_0805_2012Metric_Pad1.20x1.40mm_HandSolder
- SW1: footprint (none) -> Button_Switch_THT:SW_DIP_SPSTx02_Slide_9.78x7.26mm_W7.62mm_P2.54mm
- SW2: footprint (none) -> Button_Switch_THT:SW_Tactile_SPST_Angled_PTS645Vx31-2LFS
Connections:
- net +12V: now also J2.1 (Pin_1), J2.2 (Pin_2), J4.4 (Pin_4)
- net GNDREF: now also J2.3 (Pin_3), J4.1 (Pin_1)
- no-connect marks 0 -> 2
Other:
- note added: "ASP"
- note removed: "SPI"
- moved on the sheet: C2, C3, D2, J1, SW2, U3

Commit message: Update PCB FLicker Halogen
Parts:
- removed C1, C2, C3: 100nF, Capacitor_SMD:C_0805_2012Metric_Pad1.18x1.45mm_HandSolder, symbol Device:C
- removed SW2: SW_Push, Button_Switch_THT:SW_Tactile_SPST_Angled_PTS645Vx31-2LFS, symbol Switch:SW_Push
- removed U1: ATtiny13A-S, Package_SO:SOIC-8W_5.3x5.3mm_P1.27mm, symbol MCU_Microchip_ATtiny:ATtiny13A-S
- added J3: SW_ON, Connector_PinSocket_2.54mm:PinSocket_1x02_P2.54mm_Vertical, symbol Connector:Conn_01x02_Pin
- added U4: ATtiny13A-P, Package_DIP:DIP-8_W7.62mm, symbol MCU_Microchip_ATtiny:ATtiny13A-P
- D2: footprint Diode_SMD:D_SMB-SMC_Universal_Handsoldering -> Diode_SMD:D_SMA-SMB_Universal_Handsoldering
Connections:
- net +5V: now also J3.2 (Pin_2), U4.8 (VCC)
- net CON: now also U4.2 (PB3)
- net GND: now also U4.4 (GND)
- net MISO: now also U4.6 (PB1)
- net MOSI: now also U4.5 (PB0)
- net NRST: now also U4.1 (~{RESET}/PB5)
- net SCK: now also U4.7 (PB2)
- net SEL: now also U4.3 (PB4)
- net at U3.2 (VO): now also J3.1 (Pin_1)

Commit message: Halogen and ATTiny is hard
Parts:
- R1: value 100 -> 10K
Changed lines of the file:
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@@
     (fill (type none))
+  )
+  (text_box "Use 7805 !!!"
+    (at 85.09 96.52 0) (size 15.24 3.81)
+    (stroke (width 0) (type default))
+    (fill (type none))
+    (effects (font (size 1.27 1.27)) (justify left top))
+  )
+  (text_box "Add pull-up R\nfor NRST !!!"
+    (at 20.32 20.32 0) (size 16.51 6.35)
+    (stroke (width 0) (type default))
+    (fill (type none))
+    (effects (font (size 1.27 1.27)) (justify left top))
   )
   (text "HALOGEN CONTROL" (at 76.2 46.99 0)
@@
       (effects (font (size 1.27 1.27)))
     )
-    (property "Value" "100" (at 90.17 34.29 90)
-      (effects (font (size 1.27 1.27)))
-    )
+    (property "Value" "10K" (at 90.17 34.29 90)
+      (effects (font (size 1.27 1.27)))
+    )

Commit message: Halogen Control is On
Parts:
- R1: value 10K -> 560
Other:
- moved on the sheet: D2, J2, J3, J4, U3
