File: wira/lampu2an/lampu_v1/lampu_v1/lampu_v1.kicad_pcb (KiCad board)
At the start: 2 copper layers, 77 x 85.9 mm, 31 parts, among them J1 Conn_01x15_Pin, J10 FET, J11 Conn_01x03_Pin, J12 Conn_01x03_Pin, J13 Conn_01x03_Pin, J14 OUT1, J15 OUT2, J16 OUT3, J17 OUT4, J2 Conn_01x15_Pin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

Commit message: Lampunya Wira
Parts:
- J11: value Conn_01x03_Pin -> 3V3
- J12: value Conn_01x03_Pin -> 5V
- J13: value Conn_01x03_Pin -> GND
- JP1: moved to B.Cu
- moved J13 186.0 mm to (63.8, 36.2), turned to 90 degrees
- moved D2 185.1 mm to (74.2, 35.9)
- moved D1 180.9 mm to (74.1, 43.5)
- moved J12 180.3 mm to (63.9, 40.4), turned to 90 degrees
- moved J7 179.5 mm to (72.2, 31.2), turned to -90 degrees
- moved J11 174.7 mm to (63.8, 44.5), turned to 90 degrees
- moved R2 151.7 mm to (102.0, 33.9), turned to 180 degrees
- moved R1 149.0 mm to (102.0, 42.5), turned to 180 degrees
- moved U3 148.9 mm to (111.4, 33.7), turned to 180 degrees
- moved U2 143.8 mm to (111.5, 42.1), turned to 180 degrees
- moved JP1 140.5 mm to (97.8, 40.5), turned to -90 degrees
- moved C4 134.4 mm to (99.2, 28.6)
- moved J9 125.4 mm to (119.9, 21.5)
- moved J4 122.9 mm to (64.9, 54.2), turned to 0 degrees
- moved J17 120.1 mm to (128.2, 51.1), turned to 90 degrees
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Connections:
- R1 pad 1: +5V -> VIN
Routing:
- net P22: track 0.00 -> 128.5 mm
- net P23: track 0.00 -> 118.7 mm
- net VDD: track 0.00 -> 107.8 mm
- net P29: track 0.00 -> 97.0 mm
- net P30: track 0.00 -> 85.2 mm
- net +VDC: track 0.00 -> 72.1 mm
- net +12V: track 0.00 -> 67.0 mm, vias 0 -> 2
- net GND: track 0.00 -> 66.3 mm
- net +5V: track 0.00 -> 52.1 mm
- net VIN: track 0.00 -> 34.0 mm
- net Net-(D2-A): track 0.00 -> 18.4 mm
- net Net-(D1-A): track 0.00 -> 18.2 mm
- net P2: track 0.00 -> 11.5 mm
- net P8: track 0.00 -> 11.5 mm
- net P7: track 0.00 -> 11.5 mm
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- added copper zone on B.Cu, net GND
Other:
- board size 77 x 85.9 mm -> 77 x 86 mm
- board text added: "12V"
- board text added: "3V3"
- board text added: "5V"
- board text added: "DCIN"
- board text added: "FAN"
- board text added: "FET"
- board text added: "G"
- board text added: "GND"
- board text added: "IO0"
- board text added: "IO1"
- board text added: "IO5"
- board text added: "IO6"
- board text added: "LED-12V"
- board text added: "LED-5V"
- board text added: "PSU"
- board text added: "V+"

Commit message: Lampunya Wira
Parts:
- moved R2 14.5 mm to (87.4, 34.0)
- moved JP1 13.9 mm to (84.0, 40.0)
- moved R1 13.9 mm to (88.1, 42.0)
- moved C2 7.65 mm to (100.7, 42.5), turned to 90 degrees
- moved C3 4.63 mm to (117.5, 43.0), turned to 90 degrees
Routing:
- net +12V: track 67.0 -> 113.8 mm, vias 2 -> 0
- net Net-(D2-A): track 18.4 -> 3.83 mm
- net Net-(D1-A): track 18.2 -> 4.50 mm
- net +5V: track 52.1 -> 44.6 mm, vias 0 -> 2
- net +VDC: track 72.1 -> 78.9 mm
- net VIN: track 34.0 -> 35.8 mm

Commit message: Lampunya Wira
Other:
- board text added: "NODEMCU ESP8266"
- board text added: "USB"
Changed lines of the file:
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@@
     (effects (font (size 1 1) (thickness 0.15)) (justify left bottom))
+  )
+  (gr_text "USB" (at 85.1 50.7) (layer "F.SilkS")
+    (effects (font (size 1.5 1.5) (thickness 0.3) bold) (justify left bottom))
   )
   (gr_text "G" (at 120.8 63.9 90) (layer "F.SilkS")
@@
     (effects (font (size 1 1) (thickness 0.15)) (justify left bottom))
   )
+  (gr_text "NODEMCU ESP8266" (at 88 88.65 90) (layer "F.SilkS")
+    (effects (font (size 1.5 1.5) (thickness 0.3) bold) (justify left bottom))
+  )
   (gr_text "5V" (at 60.1 40.95) (layer "F.SilkS")
